Commit message: Fix Red Commit

File: description/lidar.xacro (robot description, xacro)
@@ -23,7 +23,8 @@
     </link>
     <gazebo reference="laser_frame">
-        <material>Gazebo/Red</material>
+        <material>Gazebo/Orange</material>
         <sensor name="laser" type="ray">
             <pose> 0 0 0 0 0 0 </pose>
+            <always_on>true</always_on>
             <visualize>true</visualize>
             <update_rate>10</update_rate>

Commit message: Update lidar.xacro

File: description/lidar.xacro (robot description, xacro)
@@ -11,5 +11,5 @@
                 <cylinder radius="0.05" length="0.04"/>
             </geometry>
-            <material name="red"/>
+            <material name="orange"/>
         </visual>
         <collision>
